File: Circuit/MCU Module/MCU_Module V3.brd (EAGLE design)
At the start: 89 x 67.5 mm, 47 parts, among them IC1 75176BD, Q1 8MHZ, T1 BC848

Commit message: finished main task for mcu
Parts:
- R12, R9: value 120 -> 75
Changed lines of the file:
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@@
 <element name="R7" library="rcl" package="R0805" value="120" x="70.29" y="43.09" rot="R90"/>
 <element name="R8" library="resistor" package="R0805" value="2k" x="65.04" y="28.31"/>
-<element name="R9" library="rcl" package="R0805" value="120" x="65.06" y="35.84"/>
+<element name="R9" library="rcl" package="R0805" value="75" x="65.06" y="35.84"/>
 <element name="RED" library="led" package="SML1206" value="" x="29.94" y="7.14"/>
 <element name="SERVO" library="pinhead" package="1X03" value="SERVO" x="70.61" y="29.48" rot="R270"/>
@@
 </element>
 <element name="R11" library="resistor" package="R0805" value="2k" x="65.15" y="41.16"/>
-<element name="R12" library="rcl" package="R0805" value="120" x="65.16" y="48.79"/>
+<element name="R12" library="rcl" package="R0805" value="75" x="65.16" y="48.79"/>
 <element name="R13" library="pot" package="B25P" value="5k" x="51.46" y="6.61" rot="R180"/>
 <element name="TRIM" library="pinhead" package="1X02" value="" x="58.27" y="10" rot="R90"/>
