File: Circuit/MCU Module/MCU_Module V3.sch (EAGLE design)
At the start: 44 parts, among them IC1 75176BD, Q1 8MHZ, T1 BC848

Commit message: finished main task for mcu
Parts:
- R12, R9: value 120 -> 75
Changed lines of the file:
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@@
 <part name="R8" library="resistor" deviceset="R-US_" device="R0805" value="2k"/>
 <part name="GND9" library="supply1" deviceset="GND" device=""/>
-<part name="R9" library="rcl" deviceset="R-US_" device="R0805" value="120"/>
+<part name="R9" library="rcl" deviceset="R-US_" device="R0805" value="75"/>
 <part name="R10" library="resistor" deviceset="R-US_" device="R0805" value="120"/>
 <part name="U$2" library="RepRapjr" deviceset="A4983CARRIER" device=""/>
@@
 <part name="R11" library="resistor" deviceset="R-US_" device="R0805" value="2k"/>
 <part name="GND17" library="supply1" deviceset="GND" device=""/>
-<part name="R12" library="rcl" deviceset="R-US_" device="R0805" value="120"/>
+<part name="R12" library="rcl" deviceset="R-US_" device="R0805" value="75"/>
 <part name="R13" library="pot" deviceset="TRIM_EU-" device="B25P" value="5k"/>
 <part name="TRIM" library="pinhead" deviceset="PINHD-1X2" device=""/>

Commit message: lots of updates
too many to document I've been a lazy uploader
Other:
- note added: "RS485 DIFFERENTIAL BUS TRANSCEIVER"
- note removed: "RS485 BUS TRANSIEVER"
Changed lines of the file:
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@@
 <text x="48" y="58" size="1.778" layer="94">multiple needs of the vending machine</text>
 <text x="103" y="64" size="2.54" layer="94">Baden David Morgan</text>
-<text x="50.8" y="182.88" size="1.778" layer="91">RS485 BUS TRANSIEVER</text>
+<text x="50.8" y="182.88" size="1.778" layer="91">RS485 DIFFERENTIAL BUS TRANSCEIVER</text>
 <text x="-99.06" y="142.24" size="1.778" layer="91" rot="R90">SERVO HEADER</text>
 <text x="-50.8" y="96.52" size="1.778" layer="91">VIBRATION MOTOR HEADER</text>
 <text x="-83.82" y="96.52" size="1.778" layer="91">INDICATOR LEDS</text>
 <text x="-66.04" y="165.1" size="1.778" layer="91" rot="R90">ADRESS SELECTOR</text>
-<text x="22.86" y="86.36" size="1.778" layer="91">GAP SENSOR HEADERS</text>
-<text x="22.86" y="83.82" size="1.778" layer="91">GAP SENSOR IS AN IR LED AND PHOTOTRANSITOR</text>
+<text x="55.88" y="86.36" size="1.778" layer="91">GAP SENSOR HEADERS</text>
+<text x="40.64" y="83.82" size="1.778" layer="91">GAP SENSOR IS AN IR LED AND PHOTOTRANSITOR</text>
 <text x="101.6" y="160.02" size="1.778" layer="91" rot="R270">LINE TERMINATION</text>
 <text x="-55.88" y="55.88" size="1.778" layer="91">STEPPER MOTOR DRIVER</text>
