File: Circuit/LCD Board/LCD_Breakout.brd (EAGLE design)
At the start: 160 x 100 mm, 4 parts, among them J1 22-05-7088-08

Commit message: lots of updates
too many to document I've been a lazy uploader
Parts:
- J1: value 22-05-7088-08 -> INTERFACE
Other:
- board size 160 x 100 mm -> 48.2 x 32.7 mm
Changed lines of the file:
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@@
 <board>
 <plain>
-<wire x1="0" y1="0" x2="160" y2="0" width="0" layer="20"/>
-<wire x1="160" y1="0" x2="160" y2="100" width="0" layer="20"/>
-<wire x1="160" y1="100" x2="0" y2="100" width="0" layer="20"/>
-<wire x1="0" y1="100" x2="0" y2="0" width="0" layer="20"/>
+<wire x1="15.24" y1="26.67" x2="63.48" y2="26.67" width="0" layer="20"/>
+<wire x1="63.48" y1="26.67" x2="63.48" y2="59.36" width="0" layer="20"/>
+<wire x1="63.48" y1="59.36" x2="15.24" y2="59.36" width="0" layer="20"/>
+<wire x1="15.24" y1="59.36" x2="15.24" y2="26.67" width="0" layer="20"/>
 <text x="36.83" y="34.29" size="1.778" layer="16" rot="MR270">GND</text>
 <text x="39.37" y="34.29" size="1.778" layer="16" rot="MR270">5V</text>
@@
 <text x="52.07" y="34.29" size="1.778" layer="16" rot="MR270">D6</text>
 <text x="54.61" y="34.29" size="1.778" layer="16" rot="MR270">D7</text>
+<dimension x1="15.24" y1="59.36" x2="15.24" y2="26.67" x3="12.7" y3="43.015" textsize="1.778" layer="20"/>
+<dimension x1="15.24" y1="26.67" x2="63.48" y2="26.67" x3="39.36" y3="22.86" textsize="1.778" layer="20"/>
 </plain>
 <attributes>
@@
 </autorouter>
 <elements>
-<element name="J1" library="con-molex" package="7395-08" value="22-05-7088-08" x="45.72" y="48.26">
+<element name="J1" library="con-molex" package="7395-08" value="INTERFACE" x="45.72" y="48.26">
 <attribute name="MPN" value="" x="45.72" y="48.26" size="1.778" layer="27" display="off"/>
 <attribute name="MF" value="" x="45.72" y="48.26" size="1.778" layer="27" display="off"/>
