File: Circuit/LCD Board/LCD_Breakout.sch (EAGLE design)
At the start: 4 parts, among them J1 22-05-7088-08

Commit message: lots of updates
too many to document I've been a lazy uploader
Parts:
- J1: value 22-05-7088-08 -> INTERFACE
Other:
- note added: "An LCD Breakout Board to make interfacing\"
- note added: "Baden Morgan"
- note added: "with the LCD easier"
Changed lines of the file:
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@@
 <setting verticaltext="up"/>
 </settings>
-<grid distance="0.1" unitdist="inch" unit="inch" style="lines" multiple="1" display="no" altdistance="0.01" altunitdist="inch" altunit="inch"/>
+<grid distance="0.1" unitdist="mm" unit="mm" style="lines" multiple="1" display="no" altdistance="0.01" altunitdist="inch" altunit="inch"/>
 <layers>
 <layer number="1" name="Top" color="4" fill="1" visible="no" active="no"/>
@@
 <part name="GND1" library="supply1" deviceset="GND" device=""/>
 <part name="R1" library="pot" deviceset="TRIM_EU-" device="CA6V" value="10k"/>
-<part name="J1" library="con-molex" deviceset="22-?-08" device="05-7088" value="22-05-7088-08"/>
+<part name="J1" library="con-molex" deviceset="22-?-08" device="05-7088" value="INTERFACE"/>
 <part name="C1" library="capacitor-wima" deviceset="C" device="5/2.5"/>
+<part name="FRAME1" library="frames" deviceset="DINA5_L" device=""/>
 </parts>
 <sheets>
 <sheet>
 <plain>
+<text x="102.9" y="-20.5" size="2.54" layer="94">Baden Morgan</text>
+<text x="48.1" y="-18.9" size="1.9304" layer="94">An LCD Breakout Board to make interfacing\</text>
+<text x="48.1" y="-21.4" size="1.9304" layer="94">with the LCD easier</text>
 </plain>
 <instances>
@@
 <instance part="J1" gate="-8" x="27.94" y="5.08" rot="R270"/>
 <instance part="C1" gate="G$1" x="81.28" y="20.32" rot="R180"/>
+<instance part="FRAME1" gate="G$1" x="-38.1" y="-40.64"/>
 </instances>
 <busses>
