File: Circuit/Power Board/Power Board V3.brd (EAGLE design)
At the start: 66.5 x 60 mm, 17 parts, among them IC1 75176AD

Commit message: lots of updates
too many to document I've been a lazy uploader
Other:
- board text added: "Power Pi Hat V1"
- board text removed: "Power Pi Hat V2"
Changed lines of the file:
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@@
 <text x="16.51" y="31.02" size="1.016" layer="21">B</text>
 <text x="46.5" y="44" size="1.778" layer="25">MRGBAD001</text>
-<text x="46.5" y="46.5" size="1.778" layer="25">Power Pi Hat V2</text>
+<text x="46.5" y="46.5" size="1.778" layer="25">Power Pi Hat V1</text>
 <text x="46.5" y="41.5" size="1.778" layer="25">UCT 2016</text>
 <dimension x1="0" y1="60" x2="0" y2="0" x3="-8" y3="30" textsize="1.778" layer="27"/>
 <dimension x1="66.5" y1="60" x2="0" y2="60" x3="33.25" y3="63.5" textsize="1.778" layer="27"/>
+<dimension x1="0" y1="60" x2="0" y2="0" x3="-4" y3="30" textsize="1.778" layer="20"/>
+<dimension x1="66.5" y1="60" x2="0" y2="60" x3="33.25" y3="-3.2" textsize="1.778" layer="20"/>
 </plain>
 <attributes>
