File: Circuit/Power Board/Power Board V3.sch (EAGLE design)
At the start: 14 parts, among them IC1 75176AD

Commit message: lots of updates
too many to document I've been a lazy uploader
Changed lines of the file:
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@@
 <part name="PI_HAT" library="con-lsta" deviceset="FE20-2" device=""/>
 <part name="R2" library="resistor" deviceset="R-US_" device="R0805" value="120"/>
-<part name="FRAME1" library="frames" deviceset="A4L-LOC" device=""/>
 <part name="R3" library="rcl" deviceset="R-US_" device="0817/7V" value="10"/>
 <part name="R4" library="rcl" deviceset="R-US_" device="0817/7V" value="10"/>
@@
 <part name="R6" library="resistor" deviceset="R-US_" device="R0805" value="2k"/>
 <part name="R7" library="resistor" deviceset="R-US_" device="R0805" value="3k6"/>
+<part name="FRAME2" library="frames" deviceset="DINA5_L" device=""/>
 </parts>
 <sheets>
 <sheet>
 <plain>
-<text x="128.27" y="-53.594" size="2.54" layer="94">Baden David Morgan</text>
-<text x="73.406" y="-52.578" size="1.778" layer="94">A Pi Hat that will function as the base for</text>
-<text x="73.152" y="-55.626" size="1.778" layer="94">the connection for power and communication</text>
-<text x="73.152" y="-58.42" size="1.778" layer="94">between the modules and the Pi itself</text>
+<text x="90.17" y="-33.274" size="2.54" layer="94">Baden David Morgan</text>
+<text x="35.306" y="-32.258" size="1.778" layer="94">A Pi Hat that will function as the base for</text>
+<text x="35.052" y="-35.306" size="1.778" layer="94">the connection for power and communication</text>
+<text x="35.052" y="-38.1" size="1.778" layer="94">between the modules and the Pi itself</text>
 </plain>
 <instances>
@@
 <instance part="PI_HAT" gate="G$1" x="2.54" y="-5.08" rot="R90"/>
 <instance part="R2" gate="G$1" x="106.68" y="0" rot="R90"/>
-<instance part="FRAME1" gate="G$1" x="-88.9" y="-73.66"/>
 <instance part="R3" gate="G$1" x="17.78" y="38.1" rot="R90"/>
 <instance part="R4" gate="G$1" x="25.4" y="38.1" rot="R90"/>
@@
 <instance part="R6" gate="G$1" x="48.26" y="-5.08" rot="R180"/>
 <instance part="R7" gate="G$1" x="43.18" y="-12.7" rot="R270"/>
+<instance part="FRAME2" gate="G$1" x="-50.8" y="-53.34"/>
 </instances>
 <busses>
